File: kischematic/kischematic.kicad_pcb (KiCad board)
At the start: 2 copper layers, 26.7 x 50 mm, 104 parts, among them IC1 BlueNRG, IC10 128x64OLED, IC2 EFM32ZG108, IC3 BQ297xx, IC4 AAT3672IWO-4.2-1, IC5 TPS6223xx, IC6 APDS-9303, IC7 APDS-9303, IC8 BSD840NH6327XTSA1, IC9 MMA8653FC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

Commit message: Getting there with the routing...
Routing:
- net DISPLAY_RESET: track 0.00 -> 4.27 mm
Changed lines of the file:
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@@
     (thickness 1.6)
     (drawings 22)
-    (tracks 1912)
+    (tracks 1920)
     (zones 0)
     (modules 104)
@@
   (segment (start 94.92 44.11) (end 95.89 45.08) (width 0.2) (layer F.Cu) (net 1) (status 30))
   (segment (start 94 47) (end 95 48) (width 0.2) (layer F.Cu) (net 1) (status 30))
+  (via (at 90.33 47.6) (size 0.62) (drill 0.31) (layers F.Cu B.Cu) (net 2))
+  (segment (start 90.33 47.6) (end 90.33 47.27) (width 0.29) (layer F.Cu) (net 2))
+  (segment (start 90.33 47.27) (end 90.388909 47.211091) (width 0.29) (layer F.Cu) (net 2))
+  (segment (start 90.33 47.6) (end 90.59 47.86) (width 0.29) (layer B.Cu) (net 2))
+  (segment (start 90.59 47.86) (end 91.81 47.86) (width 0.29) (layer B.Cu) (net 2))
   (via (at 90.65 45.52) (size 0.7) (drill 0.35) (layers F.Cu B.Cu) (net 2))
   (segment (start 90.65 45.52) (end 90.65 46.95) (width 0.29) (layer F.Cu) (net 2))
@@
   (segment (start 88.59 47.69) (end 89.37 46.91) (width 0.29) (layer F.Cu) (net 2))
   (segment (start 90.087818 46.91) (end 90.388909 47.211091) (width 0.29) (layer F.Cu) (net 2))
-  (segment (start 90.401091 47.211091) (end 90.388909 47.211091) (width 0.29) (layer F.Cu) (net 2))
-  (segment (start 90.64 47.45) (end 90.401091 47.211091) (width 0.29) (layer F.Cu) (net 2))
-  (segment (start 90.64 47.45) (end 91.05 47.86) (width 0.29) (layer B.Cu) (net 2))
-  (segment (start 91.05 47.86) (end 91.81 47.86) (width 0.29) (layer B.Cu) (net 2))
-  (via (at 90.64 47.45) (size 0.62) (drill 0.31) (layers F.Cu B.Cu) (net 2))
   (via (at 91.81 47.86) (size 0.62) (drill 0.31) (layers F.Cu B.Cu) (net 2))
   (segment (start 91.81 47.86) (end 91.74 47.86) (width 0.29) (layer F.Cu) (net 2))
@@
   (segment (start 83.9 40.7) (end 83.9 39.8) (width 0.29) (layer F.Cu) (net 102))
   (segment (start 83.95 39.75) (end 84.875 39.75) (width 0.29) (layer F.Cu) (net 102) (status 20))
+  (segment (start 90.7 48.3) (end 91.25 48.85) (width 0.16) (layer F.Cu) (net 105))
+  (segment (start 90.7 48.01) (end 90.7 48.3) (width 0.16) (layer F.Cu) (net 105))
+  (segment (start 90.78 47.93) (end 90.7 48.01) (width 0.16) (layer F.Cu) (net 105))
+  (segment (start 90.78 47.91) (end 90.78 47.93) (width 0.16) (layer F.Cu) (net 105))
+  (segment (start 91.2 47.49) (end 90.78 47.91) (width 0.16) (layer F.Cu) (net 105))
+  (segment (start 91.2 46.47) (end 91.2 47.49) (width 0.16) (layer F.Cu) (net 105))
+  (segment (start 92.083185 45.586815) (end 91.2 46.47) (width 0.16) (layer F.Cu) (net 105))
+  (segment (start 92.083185 45.381282) (end 92.083185 45.586815) (width 0.16) (layer F.Cu) (net 105))
   (segment (start 92.083185 46.618718) (end 92.071282 46.618718) (width 0.2) (layer F.Cu) (net 106))
   (zone (net 1) (net_name GND) (layer F.Cu) (hatch edge 0.508)

Commit message: Further routing tweaks.
Connections:
- P8 pad 3: SPI_CLK -> DISPLAY_RESET
- P8 pad 5: DISPLAY_RESET -> SPI_CLK
Routing:
- net SPI_CLK: track 49.1 -> 47.6 mm
Changed lines of the file:
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@@
     (thickness 1.6)
     (drawings 22)
-    (tracks 1920)
+    (tracks 1921)
     (zones 0)
     (modules 104)
@@
       (net 107 "Net-(P8-Pad6)"))
     (pad 5 smd rect (at 1 0 180) (size 0.2 0.9) (layers F.Cu F.Paste F.Mask)
-      (net 105 DISPLAY_RESET))
+      (net 31 SPI_CLK))
     (pad 4 smd rect (at 0.5 0 180) (size 0.2 0.9) (layers F.Cu F.Paste F.Mask)
       (net 106 DISPLAY_CS))
@@
       (net 30 SPI_MISO))
     (pad 3 smd rect (at 0 0 180) (size 0.2 0.9) (layers F.Cu F.Paste F.Mask)
-      (net 31 SPI_CLK))
+      (net 105 DISPLAY_RESET))
   )
   (module Capacitors_SMD:C_0402 (layer F.Cu)
@@
   (segment (start 77.8 61.3) (end 78.05 61.55) (width 0.2) (layer F.Cu) (net 30) (status 10))
   (segment (start 80.12 61.55) (end 80.8 62.23) (width 0.18) (layer F.Cu) (net 30) (status 20))
-  (segment (start 90.46 51.81) (end 91.79 51.81) (width 0.16) (layer F.Cu) (net 31))
-  (segment (start 91.79 51.81) (end 92.43 52.45) (width 0.16) (layer F.Cu) (net 31))
-  (segment (start 90.22 51.57) (end 90.46 51.81) (width 0.16) (layer F.Cu) (net 31))
-  (segment (start 90.22 51.06) (end 90.22 51.57) (width 0.16) (layer F.Cu) (net 31))
+  (segment (start 92.3 52.32) (end 92.3 50.29) (width 0.2) (layer F.Cu) (net 31))
+  (segment (start 91.53 50.3) (end 92.29 50.3) (width 0.16) (layer F.Cu) (net 31))
+  (segment (start 92.3 50.29) (end 92.3 49.79) (width 0.2) (layer F.Cu) (net 31))
+  (segment (start 92.29 50.3) (end 92.3 50.29) (width 0.16) (layer F.Cu) (net 31))
+  (segment (start 91.22 50.61) (end 91.53 50.3) (width 0.16) (layer F.Cu) (net 31))
+  (segment (start 91.22 51.06) (end 91.22 50.61) (width 0.16) (layer F.Cu) (net 31))
   (segment (start 92.43 52.45) (end 92.43 52.54) (width 0.2) (layer B.Cu) (net 31))
   (segment (start 92.43 52.54) (end 90.84 54.13) (width 0.2) (layer B.Cu) (net 31))
@@
   (segment (start 92.3 49.79) (end 93.21 48.88) (width 0.2) (layer F.Cu) (net 31))
   (segment (start 92.43 52.45) (end 92.3 52.32) (width 0.2) (layer F.Cu) (net 31))
-  (segment (start 92.3 52.32) (end 92.3 49.79) (width 0.2) (layer F.Cu) (net 31))
   (segment (start 81.12 69.5) (end 84.36 69.5) (width 0.16) (layer F.Cu) (net 31) (status 20))
   (segment (start 84.36 69.5) (end 84.62 69.24) (width 0.16) (layer F.Cu) (net 31) (status 30))
