File: kischematic/kischematic.kicad_pcb (KiCad board)
At the start: 2 copper layers, 26.7 x 50 mm, 105 parts, among them IC1 BlueNRG, IC10 128x64OLED, IC11 BALF-BRG-01D3, IC12 MAX44009, IC2 EFM32ZG108, IC3 BQ297xx, IC4 AAT3672IWO-4.2-1, IC5 TPS6223xx, IC6 MAX44009, IC8 BSD840NH6327XTSA1, IC9 MMA8653FC, J1 0, J2 Screw_Terminal_1x01, J5 Screw_Terminal_1x01, J6 Screw_Terminal_1x01, P1 CONN_01X01, P2 CONN_01X01, P3 CONN_01X01, P4 CONN_01X01, P5 CONN_01X01, P6 CONN_01X01, P7 CONN_01X01, P8 CONN_01X04, P9 CONN_01X04, SW1 SW_Push, SW2 SW_Push, U1 USB-C, U2 SWD_SPRING, U3 FT200XD, Y1 32k, Y2 16M

Commit message: Some layout improvements.
Parts:
- moved C54 5.96 mm to (86.3, 34.5)
- moved C34 0.12 mm to (87.2, 36.8)
Routing:
- net BAT+: track 31.7 -> 23.6 mm
- net GND: track 426.5 -> 427.9 mm, vias 149 -> 148
- net VUSB: track 37.1 -> 37.5 mm, vias 4 -> 2
Changed lines of the file:
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@@
     (thickness 1.6)
     (drawings 223)
-    (tracks 2205)
+    (tracks 2203)
     (zones 0)
     (modules 105)
@@
   )
   (setup
-    (last_trace_width 0.16)
+    (last_trace_width 0.2)
     (user_trace_width 0.16)
     (user_trace_width 0.2)
@@
   )
   (module Capacitors_SMD:C_0402 (layer F.Cu)
-    (at 87.26 40.41 270)
+    (at 86.325 34.52 270)
     (descr "Capacitor SMD 0402, reflow soldering, AVX (see smccp.pdf)")
     (tags "capacitor 0402")
@@
   )
   (module Capacitors_SMD:C_0402 (layer F.Cu)
-    (at 87.16 36.72 270)
+    (at 87.16 36.845 270)
     (descr "Capacitor SMD 0402, reflow soldering, AVX (see smccp.pdf)")
     (tags "capacitor 0402")
@@
   (segment (start 87.29 68.86) (end 87.3 68.85) (width 0.29) (layer B.Cu) (net 0))
   (segment (start 93.5 31.79) (end 93.61 31.68) (width 0.29) (layer B.Cu) (net 0))
+  (segment (start 86.35 36.02) (end 86.35 35.095) (width 0.2) (layer F.Cu) (net 1))
+  (segment (start 86.35 35.095) (end 86.325 35.07) (width 0.2) (layer F.Cu) (net 1))
+  (segment (start 87.16 36.295) (end 86.625 36.295) (width 0.2) (layer F.Cu) (net 1))
+  (segment (start 86.625 36.295) (end 86.35 36.02) (width 0.2) (layer F.Cu) (net 1))
+  (via (at 86.35 36.02) (size 0.7) (drill 0.35) (layers F.Cu B.Cu) (net 1))
+  (segment (start 86.325 35.07) (end 86.81 35.07) (width 0.29) (layer F.Cu) (net 1))
+  (segment (start 86.81 35.07) (end 87.19 35.45) (width 0.29) (layer F.Cu) (net 1))
   (segment (start 99.95 27.47) (end 99.375 28.045) (width 0.16) (layer F.Cu) (net 1))
   (segment (start 99.375 28.045) (end 98.85 28.045) (width 0.16) (layer F.Cu) (net 1))
@@
   (segment (start 100.85 27.47) (end 100.85 28.57) (width 0.16) (layer F.Cu) (net 1))
   (segment (start 91.1 27.2) (end 91.1 25.91) (width 0.29) (layer B.Cu) (net 1))
-  (via (at 86.76 40.78) (size 0.7) (drill 0.35) (layers F.Cu B.Cu) (net 1))
-  (segment (start 86.76 40.78) (end 86.94 40.96) (width 0.29) (layer F.Cu) (net 1))
-  (segment (start 86.83 40.85) (end 86.96 40.85) (width 0.29) (layer B.Cu) (net 1))
-  (segment (start 86.94 40.96) (end 87.26 40.96) (width 0.29) (layer F.Cu) (net 1))
-  (segment (start 86.76 40.78) (end 86.83 40.85) (width 0.29) (layer B.Cu) (net 1))
   (via (at 97.65 63.37) (size 0.7) (drill 0.35) (layers F.Cu B.Cu) (net 1))
   (segment (start 97.65 63.37) (end 96.65 63.37) (width 0.16) (layer B.Cu) (net 1))
@@
   (segment (start 79.49 27.06) (end 78.68 26.25) (width 0.16) (layer F.Cu) (net 1))
   (segment (start 79.49 28.01) (end 79.49 27.06) (width 0.16) (layer F.Cu) (net 1))
-  (segment (start 87.16 36.17) (end 87.16 35.48) (width 0.2) (layer F.Cu) (net 1) (status 10))
   (segment (start 87.16 35.48) (end 87.19 35.45) (width 0.2) (layer F.Cu) (net 1))
-  (via (at 87.19 35.45) (size 0.7) (drill 0.35) (layers F.Cu B.Cu) (net 1))
   (via (at 77.51 30.75) (size 0.62) (drill 0.31) (layers F.Cu B.Cu) (net 1))
   (segment (start 77.51 30.75) (end 77.575 30.75) (width 0.2) (layer F.Cu) (net 1))
@@
   (segment (start 85.6 36.8) (end 83.62 36.8) (width 0.24) (layer F.Cu) (net 33))
   (segment (start 83.62 36.8) (end 83.61 36.79) (width 0.26) (layer F.Cu) (net 33))
+  (segment (start 87.44 37.71) (end 87.55 37.71) (width 0.2) (layer F.Cu) (net 35))
+  (segment (start 88.38 38.39) (end 87.76 38.39) (width 0.2) (layer F.Cu) (net 35))
+  (segment (start 87.55 37.71) (end 88.3925 37.71) (width 0.2) (layer F.Cu) (net 35))
+  (segment (start 87.76 38.39) (end 87.575 38.205) (width 0.2) (layer F.Cu) (net 35))
+  (segment (start 87.575 38.205) (end 87.575 37.735) (width 0.2) (layer F.Cu) (net 35))
+  (segment (start 87.575 37.735) (end 87.55 37.71) (width 0.2) (layer F.Cu) (net 35))
+  (segment (start 87.16 37.395) (end 87.16 37.43) (width 0.2) (layer F.Cu) (net 35))
+  (segment (start 87.16 37.43) (end 87.44 37.71) (width 0.2) (layer F.Cu) (net 35))
+  (segment (start 87.78 36.28) (end 87.78 36.495) (width 0.2) (layer F.Cu) (net 35))
+  (segment (start 87.78 36.495) (end 87.78 36.65) (width 0.2) (layer F.Cu) (net 35))
+  (segment (start 87.225 37.395) (end 87.78 36.84) (width 0.2) (layer F.Cu) (net 35))
+  (segment (start 87.78 36.84) (end 87.78 36.495) (width 0.2) (layer F.Cu) (net 35))
+  (segment (start 87.16 37.395) (end 87.225 37.395) (width 0.2) (layer F.Cu) (net 35))
+  (segment (start 88.65 39.08) (end 88.65 41.04) (width 0.5) (layer F.Cu) (net 35))
+  (segment (start 88.65 41.04) (end 88.66 41.05) (width 0.5) (layer F.Cu) (net 35))
   (via (at 86.37 42.1) (size 0.7) (drill 0.35) (layers F.Cu B.Cu) (net 35))
   (segment (start 86.37 42.1) (end 86.4 42.1) (width 0.29) (layer F.Cu) (net 35))
@@
   (segment (start 88.3925 36.11) (end 87.95 36.11) (width 0.2) (layer F.Cu) (net 35) (status 10))
   (segment (start 87.95 36.11) (end 87.78 36.28) (width 0.2) (layer F.Cu) (net 35))
-  (segment (start 87.78 36.28) (end 87.78 36.65) (width 0.2) (layer F.Cu) (net 35))
-  (segment (start 87.78 36.65) (end 87.16 37.27) (width 0.2) (layer F.Cu) (net 35) (status 20))
-  (segment (start 87.42 38.05) (end 87.42 37.53) (width 0.5) (layer F.Cu) (net 35))
-  (segment (start 87.42 37.53) (end 87.16 37.27) (width 0.5) (layer F.Cu) (net 35) (status 20))
-  (segment (start 87.42 38.05) (end 87.66 38.29) (width 0.5) (layer F.Cu) (net 35))
-  (segment (start 87.66 38.29) (end 87.66 38.09) (width 0.2) (layer F.Cu) (net 35))
-  (segment (start 87.66 38.09) (end 88.04 37.71) (width 0.2) (layer F.Cu) (net 35))
-  (segment (start 88.04 37.71) (end 88.3925 37.71) (width 0.2) (layer F.Cu) (net 35) (status 20))
-  (segment (start 87.76 38.39) (end 87.66 38.29) (width 0.2) (layer F.Cu) (net 35))
-  (segment (start 88.38 38.39) (end 87.76 38.39) (width 0.2) (layer F.Cu) (net 35))
   (segment (start 88.38 38.39) (end 88.38 38.1225) (width 0.2) (layer F.Cu) (net 35) (status 20))
   (segment (start 88.38 38.1225) (end 88.3925 38.11) (width 0.2) (layer F.Cu) (net 35) (status 30))
   (segment (start 88.38 38.81) (end 88.38 38.39) (width 0.5) (layer F.Cu) (net 35))
   (segment (start 88.65 39.08) (end 88.38 38.81) (width 0.5) (layer F.Cu) (net 35))
-  (segment (start 88.66 40.64) (end 88.66 39.09) (width 0.5) (layer B.Cu) (net 35))
-  (segment (start 88.66 39.09) (end 88.65 39.08) (width 0.5) (layer B.Cu) (net 35))
-  (via (at 88.65 39.08) (size 0.7) (drill 0.35) (layers F.Cu B.Cu) (net 35))
-  (via (at 88.66 40.64) (size 0.7) (drill 0.35) (layers F.Cu B.Cu) (net 35))
   (segment (start 84.88 47.55) (end 84.88 47.32) (width 0.29) (layer F.Cu) (net 35) (status 30))
   (segment (start 97.44 48.98) (end 97.44 48.83) (width 0.2) (layer B.Cu) (net 36))
@@
   (segment (start 91.79 36.11) (end 92.01 35.89) (width 0.2) (layer F.Cu) (net 39))
   (segment (start 91.3675 36.11) (end 91.79 36.11) (width 0.2) (layer F.Cu) (net 39) (status 10))
+  (segment (start 86.325 33.97) (end 87.57 33.97) (width 0.29) (layer F.Cu) (net 40))
+  (segment (start 87.57 33.97) (end 87.67 34.07) (width 0.29) (layer F.Cu) (net 40))
   (segment (start 85.2 35.3) (end 85.2 34.6) (width 0.29) (layer F.Cu) (net 40))
-  (segment (start 85.2 34.6) (end 85.53 34.27) (width 0.29) (layer F.Cu) (net 40))
-  (segment (start 85.53 34.27) (end 87.87 34.27) (width 0.29) (layer F.Cu) (net 40))
-  (segment (start 87.87 34.27) (end 88.2 34.6) (width 0.29) (layer F.Cu) (net 40))
+  (segment (start 85.2 34.6) (end 85.73 34.07) (width 0.29) (layer F.Cu) (net 40))
+  (segment (start 85.73 34.07) (end 86.225 34.07) (width 0.29) (layer F.Cu) (net 40))
+  (segment (start 86.225 34.07) (end 86.325 33.97) (width 0.29) (layer F.Cu) (net 40))
+  (segment (start 87.67 34.07) (end 88.2 34.6) (width 0.29) (layer F.Cu) (net 40))
+  (segment (start 84.82 36.2) (end 85.2 35.82) (width 0.29) (layer F.Cu) (net 40))
+  (segment (start 85.2 35.82) (end 85.2 35.3) (width 0.29) (layer F.Cu) (net 40))
+  (segment (start 84.4 36.2) (end 84.82 36.2) (width 0.29) (layer F.Cu) (net 40))
   (segment (start 81.65 37.64) (end 82.17 37.64) (width 0.29) (layer B.Cu) (net 40))
   (segment (start 82.17 37.64) (end 82.62 37.19) (width 0.29) (layer B.Cu) (net 40))
@@
   (segment (start 83.19 37.19) (end 84.18 36.2) (width 0.29) (layer B.Cu) (net 40))
   (segment (start 84.18 36.2) (end 84.4 36.2) (width 0.29) (layer B.Cu) (net 40))
-  (segment (start 87.26 39.86) (end 87.61 39.86) (width 0.29) (layer F.Cu) (net 40))
-  (segment (start 87.61 39.86) (end 87.71 39.76) (width 0.29) (layer F.Cu) (net 40))
   (via (at 92.25 38.11) (size 0.7) (drill 0.35) (layers F.Cu B.Cu) (net 40))
   (segment (start 92.25 38.11) (end 92.25 37.03) (width 0.2) (layer B.Cu) (net 40))
@@
   (segment (start 91.3675 38.11) (end 91.385 38.11) (width 0.2) (layer F.Cu) (net 40))
   (segment (start 91.385 38.11) (end 91.525 38.25) (width 0.2) (layer F.Cu) (net 40))
-  (segment (start 84.4 36.2) (end 85.69 36.2) (width 0.29) (layer F.Cu) (net 40))
-  (segment (start 85.69 36.2) (end 85.74 36.25) (width 0.29) (layer F.Cu) (net 40))
-  (segment (start 85.74 36.25) (end 85.78 36.25) (width 0.29) (layer F.Cu) (net 40))
-  (segment (start 85.78 36.25) (end 86.56 37.03) (width 0.29) (layer F.Cu) (net 40))
-  (segment (start 87.71 39.76) (end 91.27 39.76) (width 0.29) (layer F.Cu) (net 40))
-  (segment (start 86.56 37.03) (end 86.56 38.61) (width 0.29) (layer F.Cu) (net 40))
   (segment (start 91.525 39.505) (end 91.525 38.25) (width 0.29) (layer F.Cu) (net 40))
-  (segment (start 86.56 38.61) (end 87.71 39.76) (width 0.29) (layer F.Cu) (net 40))
   (segment (start 91.27 39.76) (end 91.525 39.505) (width 0.29) (layer F.Cu) (net 40))
   (via (at 84.4 36.2) (size 0.62) (drill 0.31) (layers F.Cu B.Cu) (net 40))

Commit message: Minor.
Routing:
- net (no net): track 3.73 -> 0.93 mm
Changed lines of the file:
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@@
     (thickness 1.6)
     (drawings 223)
-    (tracks 2203)
+    (tracks 2200)
     (zones 0)
     (modules 105)
@@
   (gr_line (start 76 25) (end 102.7 25) (layer Edge.Cuts) (width 0.05))
   (segment (start 88.52 55.87) (end 88.75 55.64) (width 0.16) (layer B.Cu) (net 0))
-  (segment (start 87.29 68.86) (end 87.29 66.42) (width 0.2) (layer B.Cu) (net 0))
   (segment (start 85.98 58.66) (end 85.82 59.08) (width 0.2) (layer B.Cu) (net 0))
-  (segment (start 87.3 68.85) (end 87.65 68.85) (width 0.29) (layer B.Cu) (net 0))
-  (segment (start 87.29 68.86) (end 87.3 68.85) (width 0.29) (layer B.Cu) (net 0))
   (segment (start 93.5 31.79) (end 93.61 31.68) (width 0.29) (layer B.Cu) (net 0))
   (segment (start 86.35 36.02) (end 86.35 35.095) (width 0.2) (layer F.Cu) (net 1))
