File: progconnector_schematic/progconnector.sch (KiCad schematic (older format))
At the start: 10 parts, among them J1 Screw_Terminal_1x01, J10 Screw_Terminal_1x01, J2 Screw_Terminal_1x01, J3 Screw_Terminal_1x01, J4 Screw_Terminal_1x01, J5 Screw_Terminal_1x01, J6 Screw_Terminal_1x01, J7 Screw_Terminal_1x01, J8 Screw_Terminal_1x01, J9 Screw_Terminal_1x01

Commit message: Work on programming connector board.
Parts:
- removed J1: Screw_Terminal_1x01, Pin_Headers:Pin_Header_Straight_1x01_Pitch2.54mm, symbol Screw_Terminal_1x01
- removed J6: Screw_Terminal_1x01, newlightmeter:POGOHOLDER, symbol Screw_Terminal_1x01
Connections:
- wire segments 25 -> 20
Changed lines of the file:
@@
 $EndDescr
-$Comp
-L Screw_Terminal_1x01 J1
-U 1 1 589F18FF
-P 5800 2550
-F 0 "J1" H 5720 2504 50  0000 R CNN
-F 1 "Screw_Terminal_1x01" H 5720 2595 50  0000 R CNN
-F 2 "Pin_Headers:Pin_Header_Straight_1x01_Pitch2.54mm" H 5800 2425 50  0001 C CNN
-F 3 "" H 5800 2450 50  0001 C CNN
-	1    5800 2550
-	-1   0    0    1
-$EndComp
 $Comp
 L Screw_Terminal_1x01 J2
@@
 $EndComp
 Wire Wire Line
-	4950 2550 5600 2550
-Wire Wire Line
 	4950 2900 5600 2900
 Wire Wire Line
@@
 Wire Wire Line
 	4950 4000 5600 4000
-Wire Wire Line
-	5400 2550 5400 2400
-Wire Wire Line
-	5400 2400 7200 2400
-Wire Wire Line
-	7200 2400 7200 2550
-Connection ~ 5400 2550
 Wire Wire Line
 	5400 2900 5400 2750
@@
 Connection ~ 5400 4000
 Wire Wire Line
-	7200 2550 7500 2550
-Wire Wire Line
 	7200 2900 7500 2900
 Wire Wire Line
@@
 	7200 4000 7500 4000
 $Comp
-L Screw_Terminal_1x01 J6
-U 1 1 589F1D64
-P 7700 2550
-F 0 "J6" H 7620 2504 50  0000 R CNN
-F 1 "Screw_Terminal_1x01" H 7620 2595 50  0000 R CNN
-F 2 "newlightmeter:POGOHOLDER" H 7700 2425 50  0001 C CNN
-F 3 "" H 7700 2450 50  0001 C CNN
-	1    7700 2550
-	-1   0    0    1
-$EndComp
-$Comp
 L Screw_Terminal_1x01 J7
